Commit message: 2nd ver jtc
Added the ability to select the type of paths to Qt application: Windows or Linux

File: Projekty Qt/Dane JTC/avena_arm_id.urdf (robot description, URDF)
Before this commit: robot avena, 9 links, 8 joints
Links:
- link avena_link_3: mass 3.375 -> 5.
Joints:
- joint avena_joint_3: origin xyz=-0.467 0 0.009 rpy=0 3.1415 0 -> xyz=-0.686 0 0 rpy=0 3.1415 0
- joint avena_joint_4: origin xyz=0.452 0 0.0226 rpy=3.1415 0 0 -> xyz=0.671 0 -0.005 rpy=3.1415 0 0
